Commit message: add 2 more drawers for training

File: src/urdf/custom/output/label31.urdf (robot description, URDF)
Before this commit: robot my_urdf, 7 links, 6 joints
Links:
- removed link knob3
- added link handle3, mass 0.2; collision mesh filename=../meshes/parts/handle.obj scale=1 1 1; visual mesh filename=../meshes/parts/handle.obj scale=1 1 1
Joints:
- joint knob3_to_drawer0: child knob3 -> handle3
